File: max2871-evalboard/max2871-evalboard.kicad_sch (KiCad schematic)
At the start: 15 parts

Commit message: Finish schematic - create PCB
Parts:
- removed D?: LED, LED_THT:LED_D5.0mm_Horizontal_O1.27mm_Z3.0mm, symbol Device:LED
- removed J?: Conn_02x05_Odd_Even, Connector_PinHeader_2.54mm:PinHeader_2x05_P2.54mm_Horizontal, symbol Connector_Generic:Conn_02x05_Odd_Even
- removed J?: USB_B, USB-B1HSB6:OST_USB-B1HSB6, symbol Connector:USB_B
- removed SW?: SW_Push_DPDT, symbol Switch:SW_Push_DPDT
- added D101: LED, LED_THT:LED_D3.0mm_Horizontal_O3.81mm_Z2.0mm, symbol Device:LED
- added J101: USB_B_Mini, 54819-0519:MOLEX_54819-0519, symbol Connector:USB_B_Mini
- added J103: Conn_02x06_Odd_Even, Connector_PinHeader_2.54mm:PinHeader_2x06_P2.54mm_Horizontal, symbol Connector_Generic:Conn_02x06_Odd_Even
- added SW101: XKBS22E05-Z, XKBS22E05-Z:XKBS22E05-Z, symbol XKBS22E05-Z:XKBS22E05-Z
- added TP101, TP102, TP103, TP104, TP105, TP106: (no value), TestPoint:TestPoint_Pad_D1.5mm, symbol Connector:TestPoint
- C101: renamed from C?; Partnumber (none) -> CS3225X5R476K160NRL
- C102, C103: renamed from C?; Partnumber (none) -> GCM155R71H102KA37D
- C104: renamed from C?; Partnumber (none) -> TMK105B7103KVHF
- D102, D103: renamed from D?; Partnumber (none) -> SS12
- J104, J105: renamed from J?; Partnumber (none) -> DOSIN-806-0186
- R101: renamed from R?; LCSC (none) -> C705665; Manufacturer (none) -> YAGEO; Part Number (none) -> RT0402CRE071KL; Partnumber (none) -> RT0402CRE071KL
- R102: renamed from R?; Partnumber (none) -> PTFR0402B49R9N9
- gave numbers to parts that had none: 1
Connections:
- net +5V: now also SW101.2 (B), SW101.5 (B), TP102.1
- net CE: now also J103.8 (Pin_8), TP106.1
- net DATA: now also J103.4 (Pin_4), TP104.1
- net GND: now also D101.1 (K), J101.5 (GND), J101.6 (Shield), J103.11 (Pin_11), J103.12 (Pin_12), SW101.7 (Shield)
- net PWR: now also SW101.3 (C), SW101.6 (C), TP101.1
- net SCLK: now also J103.2 (Pin_2), TP103.1
- net SPI_CLK: now also J103.1 (Pin_1)
- net SPI_CS: now also J103.7 (Pin_7)
- net SPI_DATA: now also J103.3 (Pin_3)
- net USB_D+: now also J101.3 (D+)
- net USB_D-: now also J101.2 (D-)
- net at C101.1, D103.2 (A): now also J101.1 (VBUS)
- net at R101.1: now also D101.2 (A)
- net REF_IN renamed vco/REF_IN
- new net EN_TXCO: J103.10 (Pin_10)
- new net MUX: J103.6 (Pin_6), TP105.1
- new net SPI_MISO: J103.5 (Pin_5)
- new net TXCO_PWR: J103.9 (Pin_9)
- no-connect marks 3 -> 4
Other:
- sheet vco ports: added EN_TXCO, TXCO_PWR; removed none
- note added: "This header gives the option to use an external SPI controller for the VCO. For normal operation, jumpers should be added here."
- moved on the sheet: C102, C103, C104, J104, J105, R102

Commit message: PCB placement complete
Parts:
- J102: footprint Connector_PinHeader_2.54mm:PinHeader_2x05_P2.54mm_Vertical_SMD -> Connector_PinHeader_2.54mm:PinHeader_2x05_P2.54mm_Vertical
Connections:
- net CE renamed LE
- no-connect marks 4 -> 3
Other:
- sheet microcontroller ports: added VCO_CE; removed VCO_LE, VCO_MUX
- sheet vco ports: added ~{CE}; removed CE

Commit message: Finish layout design
Parts:
- removed J101: USB_B_Mini, 54819-0519:MOLEX_54819-0519, symbol Connector:USB_B_Mini
- added J101: USB_C_Receptacle_USB2.0, USB4105-GF-A:GCT_USB4105-GF-A, symbol Connector:USB_C_Receptacle_USB2.0
- added R101, R103: DNP, Resistor_SMD:R_0402_1005Metric, symbol Device:R
- added R102, R104: 5.1k, Resistor_SMD:R_0402_1005Metric, symbol Device:R
- C101: value 47uF -> 10uF; footprint Capacitor_SMD:C_1210_3225Metric -> Capacitor_SMD:C_0603_1608Metric; LCSC C2918513 -> C92487; Manufacturer Samwha Capacitor -> Samsung; Part Number CS3225X5R476K160NRL -> CL10A106MO8NQNC; Partnumber CS3225X5R476K160NRL -> GCM155C71A105KE38D
- J103: renamed from J102; footprint Connector_PinHeader_2.54mm:PinHeader_2x05_P2.54mm_Vertical -> Connector_PinHeader_1.27mm:PinHeader_2x05_P1.27mm_Vertical
- TP101: renamed from TP103; footprint TestPoint:TestPoint_Pad_D1.5mm -> TestPoint:TestPoint_Pad_D1.0mm
- TP102: renamed from TP104; footprint TestPoint:TestPoint_Pad_D1.5mm -> TestPoint:TestPoint_Pad_D1.0mm
- TP103: renamed from TP105; footprint TestPoint:TestPoint_Pad_D1.5mm -> TestPoint:TestPoint_Pad_D1.0mm
- TP104: renamed from TP106; footprint TestPoint:TestPoint_Pad_D1.5mm -> TestPoint:TestPoint_Pad_D1.0mm
- renumbered D102 to D101, D103 to D102, D101 to D103, J103 to J102, R101 to R105, R102 to R106, TP102 to TP105, TP101 to TP106
Connections:
- net GND: now also J101.A1 (GND), J101.A12 (GND), J101.B1 (GND), J101.B12 (GND), J101.S1 (SHIELD), R102.2, R104.2
- net SWCLK: now also J103.3 (Pin_3); no longer J103.4 (Pin_4)
- net SWD: now also J103.4 (Pin_4); no longer J103.3 (Pin_3)
- net USB_D+: now also J101.A6 (D+), J101.B6 (D+)
- net USB_D-: now also J101.A7 (D-), J101.B7 (D-)
- net VBUS: now reaches C101.1, D102.2 (A)
- net VBUS: now also J101.A4 (VBUS), J101.A9 (VBUS), J101.B4 (VBUS), J101.B9 (VBUS), R101.2, R103.2
- new net: J101.A5 (CC1), R103.1, R104.1
- new net: J101.B5 (CC2), R101.1, R102.1
- no-connect marks 3 -> 4
Other:
- note added: "Power switch"
- moved on the sheet: C102, C103, C104, D102, D103, J102, J104, J105, R105, R106, SW101, TP101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
