File: max2871-evalboard/microcontroller.kicad_sch (KiCad schematic)
At the start: 35 parts

Commit message: Finish schematic - create PCB
Parts:
- removed C? (x4): 1uF, Capacitor_SMD:C_0402_1005Metric, symbol Device:C
- removed C?: 100nF, Capacitor_SMD:C_0402_1005Metric, symbol Device:C
- removed C?: 30pF, Capacitor_SMD:C_0402_1005Metric, symbol Device:C
- removed D?: LED, LED_SMD:LED_0603_1608Metric, symbol Device:LED
- removed R? (x5): 1k, Resistor_SMD:R_0402_1005Metric, symbol Device:R
- added C201, C202, C206, C217: 1uF, Capacitor_SMD:C_0402_1005Metric, symbol Device:C
- added C203: 100nF, Capacitor_SMD:C_0402_1005Metric, symbol Device:C
- added C205: 30pF, Capacitor_SMD:C_0402_1005Metric, symbol Device:C
- added D202: LED, LED_SMD:LED_0603_1608Metric, symbol Device:LED
- added Q201, Q202: 2N7002, Package_TO_SOT_SMD:SOT-23, symbol Transistor_FET:2N7002
- added R201, R202, R205, R209, R210: 1k, Resistor_SMD:R_0402_1005Metric, symbol Device:R
- added TP201, TP202, TP203, TP204, TP205, TP206: (no value), TestPoint:TestPoint_Pad_D1.5mm, symbol Connector:TestPoint
- C204: renamed from C?; LCSC (none) -> C161152; Manufacturer (none) -> Murata; Part Number (none) -> GCM1555C1H300JA16D; Partnumber (none) -> GCM1555C1H300JA16D
- C207, C208, C209, C210, C211, C212, C213, C214, C215, C216: renamed from C?; Partnumber (none) -> CL05F104ZO5NNNC
- D201: renamed from D?; LCSC (none) -> C72043; Manufacturer (none) -> Everlight; Part Number (none) -> 19-217/GHC-YR1S2/3T; Partnumber (none) -> 19-217/GHC-YR1S2/3T
- R203: renamed from R?; LCSC (none) -> C852428; Manufacturer (none) -> YAGEO; Part Number (none) -> RT0402BRC0710KL; Partnumber (none) -> RT0402BRC0710KL
- R206, R207: renamed from R?; LCSC (none) -> C31439; Manufacturer (none) -> UNI-ROYAL; Part Number (none) -> 0402WGF274JTCE; Partnumber (none) -> 0402WGF274JTCE
- SW201, SW202: renamed from SW?; Partnumber (none) -> TSA017A2540A03
- U201: renamed from U?; LCSC (none) -> C92517; Manufacturer (none) -> Diodes Inc; Part Number (none) -> AZ1117H-3.3TRE1; Partnumber (none) -> AZ1117H-3.3TRE1
- U202: renamed from U?; LCSC (none) -> C113767; Manufacturer (none) -> Winbond; Part Number (none) -> W25Q128JVSIQ; Partnumber (none) -> W25Q128JVSIQ
- U203: renamed from U?; LCSC (none) -> C2040; Manufacturer (none) -> Raspberry Pi; Part Number (none) -> RP2040; Partnumber (none) -> RP2040
- Y201: renamed from Y?; Partnumber (none) -> TAXM12M4RLBDDT2T
- gave numbers to parts that had none: 2
Connections:
- net +1V1: now also C206.1, TP205.1
- net +3V3: now also C202.1, C203.1, C217.1, R209.1, R210.1, TP203.1, TP206.1
- net GND: now also C201.2, C202.2, C203.2, C205.1, C206.2, C217.2, Q201.2 (S), Q202.2 (S), R201.1; no longer D201.1 (K)
- net QSPI_SS: now also R202.2, TP202.1
- net RESET: now also TP204.1
- net VIN: now also C201.1, TP201.1
- net at R208.1, U203.21 (XOUT): now also R205.2
- net at SW202.1: now also R201.2
- net LED1: now reaches U203.36 (GPIO24)
- net LED1: now also Q201.1 (G)
- net at Y201.1: now also C205.2, R205.1
- net LED2: now reaches U203.37 (GPIO25)
- net LED2: now also Q202.1 (G)
- net at D201.2 (A): now also R209.2
- net at SW201.2: now also R202.1
- new net: D201.1 (K), Q201.3 (D)
- new net: D202.2 (A), R210.2
- new net: D202.1 (K), Q202.3 (D)
- no-connect marks 2 -> 18
Other:
- note added: "Place R206 and R207 resistors close to pins 46 and 47"
- note removed: "Place RX and RY resistors close to pins 46 and 47"
- moved on the sheet: D201, R204

Commit message: PCB placement complete
Parts:
- removed TP201, TP203: (no value), TestPoint:TestPoint_Pad_D1.5mm, symbol Connector:TestPoint
Connections:
- net LED1: now also U203.13 (GPIO10); no longer U203.36 (GPIO24)
- net LED2: now also U203.14 (GPIO11); no longer U203.37 (GPIO25)
- net VCO_LE: no longer names the net of U203.12 (GPIO9)
- net VCO_MUX renamed VCO_CE
- no-connect marks 18 -> 19

Commit message: Finish layout design
Parts:
- added C204: 2.2uF, Capacitor_SMD:C_0402_1005Metric, symbol Device:C
- added D201: LED, LED_THT:LED_D3.0mm_Horizontal_O3.81mm_Z2.0mm, symbol Device:LED
- added Q201: 2N7002, Package_TO_SOT_SMD:SOT-23, symbol Transistor_FET:2N7002
- added R209: 1k, Resistor_SMD:R_0402_1005Metric, symbol Device:R
- C201: value 1uF -> 10uF; footprint Capacitor_SMD:C_0402_1005Metric -> Capacitor_SMD:C_0603_1608Metric; LCSC C126521 -> C92487; Manufacturer Murata -> Samsung; Part Number GCM155C71A105KE38D -> CL10A106MO8NQNC
- C202: value 1uF -> 22uF; footprint Capacitor_SMD:C_0402_1005Metric -> Capacitor_SMD:C_0805_2012Metric; LCSC C126521 -> C602037; Manufacturer Murata -> Samsung; Part Number GCM155C71A105KE38D -> CL21A226MAYNNNE
- C207: renamed from C206; Partnumber GCM155C71A105KE38D -> (none)
- C218: renamed from C217; Partnumber GCM155C71A105KE38D -> (none)
- renumbered C204 to C205, C205 to C206, C207 to C208, C208 to C209, C209 to C210, C210 to C211, C211 to C212, C212 to C213, C213 to C214, C214 to C215, C215 to C216, C216 to C217, D201 to D202, D202 to D203, Q201 to Q202, Q202 to Q203, R209 to R210, R210 to R211, TP202 to TP201, TP204 to TP202, TP205 to TP203, TP206 to TP204
Connections:
- net +3V3: now also C204.1, R209.1
- net GND: now also C204.2, Q201.2 (S)
- net LED_LOCK: now reaches U203.36 (GPIO24)
- net LED_LOCK: now also Q201.1 (G)
- new net: D201.1 (K), Q201.3 (D)
- new net: D201.2 (A), R209.2
- no-connect marks 19 -> 18
Other:
- moved on the sheet: C203, R204
